File: Sensing.kicad_sch (KiCad schematic)
At the start: 20 parts, among them Q1 ZXMP2120FFTA, Q2 ZXMP2120FFTA, U1 LTC4368CMS-1#PBF, U2 INA226AIDGSR, U3 MCP9808T-E/MS, U7 MCP9808T-E/MS, U8 MCP9808T-E/MS

Commit message: Added actuation circuit for x, y, and z axes
Parts:
- added C14, C15, C16: ${VALUE}, symbol Capacitor:Capacitor_NP
- added C17: ${VALUE}, Package_SO:Toshiba_SOIC-4-6_4.4x3.6mm_P1.27mm, symbol Capacitor:Capacitor_POL
- added Q3, Q4: ZXMP2120FFTA, Other:TRXSOFL3P95_290X240X100L58X40N, symbol DB:Transistor/348
- added R13, R14, R15, R16, R17, R18, R19, R20, R21: ${VALUE}, Other:DPAK3P508_1229X317L176X89T749X673N, symbol Resistor:Resistor
- added U10: INA226AIDGSR, Leaded:DGS10, symbol DB:Power/2606
- added U11: LTC4368CMS-1#PBF, Leaded:MS_10_ADI, symbol DB:Protection/2607
Connections:
- net *SHDN: now also R13.2, R14.1, U11.6 (*SHDN)
- net CURR_LIM_1_NFAULT: now also U11.7 (FAULT)
- net GND: now also C14.2, C15.1, C16.2, C17.2, R16.2, U10.7 (GND), U11.11 (EPAD), U11.5 (GND)
- net OV: now also R15.2, R16.1, U11.3 (OV)
- net RETRY: now also C14.1, U11.4 (RETRY)
- net UV: now also R14.2, R15.1, U11.2 (UV)
- net VBUS: no longer C4.2, Q1.2 (D), R1.1, R7.1, R8.1, R9.1, U1.1 (VIN), U2.6 (VS)
- net VOUT: now also C17.1, Q3.2 (D), R19.1, U11.8 (VOUT)
- net VSENSE_A0: now also U10.2 (A0)
- net VSENSE_A1: now also U10.1 (A1)
- net VSENSE_ALERT: now also R21.2, U10.3 (ALERT)
- net VSENSE_N: now also U10.9 (VIN-)
- net VSENSE_P: now also U10.10 (VIN+), U10.8 (VBUS)
- net VSENSE_SCL: now also R20.2, U10.5 (SCL)
- net VSENSE_SDA: now also R18.2, U10.4 (SDA)
- net TEMP1_ALERT: now reaches U3.3 (ALERT)
- net TEMP3_ALERT: now reaches U7.3 (ALERT)
- net TEMP2_ALERT: now reaches U8.3 (ALERT)
- new net: C16.1, R17.2
- new net: R19.2, U11.9 (SENSE)
- new net: Q3.1 (D), Q4.1 (D), R17.1, U11.10 (GATE)
- new net: Q3.3 (G), Q4.3 (G)
- new net VBUS_5V: C15.2, C4.2, Q1.2 (D), Q4.2 (D), R1.1, R13.1, R18.1, R20.1, R21.1, R7.1, R8.1, R9.1, U1.1 (VIN), U10.6 (VS), U11.1 (VIN), U2.6 (VS)
Other:
- note added: "Current Sensing 3.3V"
- note added: "Current Sensing 5V"
- note added: "Temperature Sensing"
- note added: "Voltage Sensing 3.3V"
- note added: "Voltage Sensing 5V"
- note removed: "Current Sensing (x2)"
- note removed: "Voltage Sensing"
- moved on the sheet: U3, U7, U8

Commit message: Added debug schematic sheet and ST-Link 14 pin header
Parts:
- added U12, U13, U14: INA226AIDGSR, Leaded:DGS10, symbol DB:Power/2606
Other:
- note added: "Current Limiting 3.3V"
- note added: "Current Limiting 5V"
- note removed: "Current Sensing 3.3V"
- note removed: "Current Sensing 5V"
